File: pcb/nabu-rs232.kicad_sch (KiCad schematic)
At the start: 30 parts, among them J1 NABU expansion slot, J2 TTL, J3 RS232, U1 74LS139, U2 74LS32, U3 74HCT04, U4 74HCT244, U5 8251, U6 74LS245, U7 8253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

Commit message: version 0.1 sent to jlcpcb
Parts:
- added J4: RS232 enable, Connector_PinHeader_2.54mm:PinHeader_2x03_P2.54mm_Vertical, symbol Connector_Generic:Conn_02x03_Odd_Even
Connections:
- net CTS: now also J4.3 (Pin_3); no longer U9.9 (R2OUT)
- net RXD: now also J4.5 (Pin_5); no longer U8.12 (R1OUT)
- net at U5.22 (~{DSR}): now also J4.1 (Pin_1); no longer U9.12 (R1OUT)
- new net: J4.2 (Pin_2), U9.12 (R1OUT)
- new net: J4.4 (Pin_4), U9.9 (R2OUT)
- new net: J4.6 (Pin_6), U8.12 (R1OUT)
Changed lines of the file:
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@@
     (company "Hans Hübner")
   )
+  (junction (at 247.142 73.406) (diameter 0) (color 0 0 0 0)
+  )
+  (junction (at 249.682 83.566) (diameter 0) (color 0 0 0 0)
+  )
+  (junction (at 302.768 186.944) (diameter 0) (color 0 0 0 0)
+  )
+  (junction (at 302.768 199.644) (diameter 0) (color 0 0 0 0)
+  )
   (junction (at 257.302 75.946) (diameter 0) (color 0 0 0 0)
-  )
-  (junction (at 247.142 73.406) (diameter 0) (color 0 0 0 0)
-  )
-  (junction (at 249.682 83.566) (diameter 0) (color 0 0 0 0)
-  )
-  (junction (at 302.768 186.944) (diameter 0) (color 0 0 0 0)
-  )
-  (junction (at 302.768 199.644) (diameter 0) (color 0 0 0 0)
   )
   (junction (at 252.222 81.026) (diameter 0) (color 0 0 0 0)
@@
     (stroke (width 0) (type default) (color 0 0 0 0))
   )
-  (wire (pts (xy 249.682 83.566) (xy 267.208 83.566))
+  (wire (pts (xy 249.682 83.566) (xy 271.78 83.566))
     (stroke (width 0) (type default) (color 0 0 0 0))
   )
@@
     (stroke (width 0) (type default) (color 0 0 0 0))
   )
+  (wire (pts (xy 257.302 75.946) (xy 276.098 75.946))
+    (stroke (width 0) (type default) (color 0 0 0 0))
+  )
   (wire (pts (xy 348.488 73.406) (xy 360.68 73.406))
     (stroke (width 0) (type default) (color 0 0 0 0))
@@
     (stroke (width 0) (type default) (color 0 0 0 0))
   )
+  (wire (pts (xy 288.798 78.486) (xy 295.656 78.486))
+    (stroke (width 0) (type default) (color 0 0 0 0))
+  )
   (wire (pts (xy 302.26 56.896) (xy 307.34 56.896))
     (stroke (width 0) (type default) (color 0 0 0 0))
@@
     (stroke (width 0) (type default) (color 0 0 0 0))
   )
-  (wire (pts (xy 267.208 73.406) (xy 307.34 73.406))
-    (stroke (width 0) (type default) (color 0 0 0 0))
-  )
   (wire (pts (xy 244.348 73.406) (xy 247.142 73.406))
     (stroke (width 0) (type default) (color 0 0 0 0))
@@
     (stroke (width 0) (type default) (color 0 0 0 0))
   )
+  (wire (pts (xy 295.656 127.762) (xy 307.086 127.762))
+    (stroke (width 0) (type default) (color 0 0 0 0))
+  )
+  (wire (pts (xy 288.798 73.406) (xy 307.34 73.406))
+    (stroke (width 0) (type default) (color 0 0 0 0))
+  )
   (wire (pts (xy 375.92 79.248) (xy 375.92 68.326))
     (stroke (width 0) (type default) (color 0 0 0 0))
@@
     (stroke (width 0) (type default) (color 0 0 0 0))
   )
-  (wire (pts (xy 267.208 83.566) (xy 267.208 127.762))
+  (wire (pts (xy 271.78 83.566) (xy 271.78 78.486))
     (stroke (width 0) (type default) (color 0 0 0 0))
   )
@@
     (stroke (width 0) (type default) (color 0 0 0 0))
   )
+  (wire (pts (xy 271.78 78.486) (xy 276.098 78.486))
+    (stroke (width 0) (type default) (color 0 0 0 0))
+  )
   (wire (pts (xy 343.916 79.248) (xy 375.92 79.248))
     (stroke (width 0) (type default) (color 0 0 0 0))
@@
     (stroke (width 0) (type default) (color 0 0 0 0))
   )
+  (wire (pts (xy 295.656 78.486) (xy 295.656 127.762))
+    (stroke (width 0) (type default) (color 0 0 0 0))
+  )
   (wire (pts (xy 336.55 60.706) (xy 346.202 60.706))
     (stroke (width 0) (type default) (color 0 0 0 0))
@@
     (stroke (width 0) (type default) (color 0 0 0 0))
   )
+  (wire (pts (xy 288.798 75.946) (xy 307.34 75.946))
+    (stroke (width 0) (type default) (color 0 0 0 0))
+  )
   (wire (pts (xy 302.006 108.712) (xy 302.006 111.252))
     (stroke (width 0) (type default) (color 0 0 0 0))
@@
     (stroke (width 0) (type default) (color 0 0 0 0))
   )
-  (wire (pts (xy 267.208 127.762) (xy 307.086 127.762))
-    (stroke (width 0) (type default) (color 0 0 0 0))
-  )
   (wire (pts (xy 345.948 117.602) (xy 345.948 135.382))
     (stroke (width 0) (type default) (color 0 0 0 0))
@@
     (stroke (width 0) (type default) (color 0 0 0 0))
   )
+  (wire (pts (xy 267.208 73.406) (xy 276.098 73.406))
+    (stroke (width 0) (type default) (color 0 0 0 0))
+  )
   (wire (pts (xy 267.208 70.866) (xy 267.208 73.406))
     (stroke (width 0) (type default) (color 0 0 0 0))
@@
   )
   (wire (pts (xy 244.348 75.946) (xy 257.302 75.946))
-    (stroke (width 0) (type default) (color 0 0 0 0))
-  )
-  (wire (pts (xy 257.302 75.946) (xy 307.34 75.946))
     (stroke (width 0) (type default) (color 0 0 0 0))
   )
@@
     )
     (pin "1")
+  )
+  (symbol (lib_id "Connector_Generic:Conn_02x03_Odd_Even") (at 281.178 75.946 0) (unit 1)
+    (in_bom yes) (on_board yes)
+    (property "Reference" "J4" (id 0) (at 282.448 81.28 0))
+    (property "Value" "RS232 enable" (id 1) (at 282.448 83.312 0))
+    (property "Footprint" "Connector_PinHeader_2.54mm:PinHeader_2x03_P2.54mm_Vertical" (id 2) (at 281.178 75.946 0)
+      (effects (font (size 1.27 1.27)) hide)
+    )
+    (property "Datasheet" "~" (id 3) (at 281.178 75.946 0)
+      (effects (font (size 1.27 1.27)) hide)
+    )
+    (pin "1")
+    (pin "2")
+    (pin "3")
+    (pin "4")
+    (pin "5")
+    (pin "6")
   )
   (symbol (lib_id "nabu-rs232:NABU option connector") (at 92.71 127.254 0) (mirror y) (unit 1)
@@
       (reference "J3") (unit 1) (value "RS232") (footprint "Connector_PinHeader_2.54mm:PinHeader_2x05_P2.54mm_Horizontal")
     )
+    (path "/0438a8ac-2098-49b9-8656-62b3bcf23182"
+      (reference "J4") (unit 1) (value "RS232 enable") (footprint "Connector_PinHeader_2.54mm:PinHeader_2x03_P2.54mm_Vertical")
+    )
     (path "/1ff44661-c156-483f-ad15-57619bf9a0e9"

Commit message: Use proper DB9 RS232 pinout
Parts:
- J3: value RS232 -> RS232 (DB9)
Connections:
- net GND: now also J3.5 (Pin_5); no longer J3.9 (Pin_9)
- net at U8.13 (R1IN): now also J3.2 (RXD); no longer J3.3 (Pin_3)
- net at U8.14 (T1OUT): now also J3.3 (TXD); no longer J3.5 (Pin_5)
- net at U9.13 (R1IN): now also J3.6 (DSR); no longer J3.2 (Pin_2)
- net at U9.14 (T1OUT): now also J3.4 (DTR); no longer J3.7 (Pin_7)
- net at U9.7 (T2OUT): now also J3.7 (RTS); no longer J3.4 (Pin_4)
- net at U9.8 (R2IN): now also J3.8 (CTS); no longer J3.6 (Pin_6)
- no-connect marks 19 -> 18
